Commit message: fix

File: test_package/xacro/bot.xacro (robot description, xacro)
@@ -6,5 +6,5 @@
       <origin xyz="0 0 0"  rpy="0 0 0"/>
       <geometry>
-        <cylinder radius=1 length=1/>
+        <cylinder radius="1" length="1"/>
       </geometry>
       <material name="grey"/>
@@ -13,5 +13,5 @@
       <origin xyz="0.0 0.0 0.0" rpy="0 0 0"/>
       <geometry>
-        <cylinder radius=1 length=1/>
+        <cylinder radius="1" length="1"/>
       </geometry>
     </collision>

Commit message: xarco

File: test_package/xacro/bot.xacro (robot description, xacro)
@@ -24,3 +24,32 @@
     </inertial>
   </link>
+  <link name="child_link">
+    <visual>
+      <origin xyz="0 0 0"  rpy="0 0 0"/>
+      <geometry>
+        <cylinder radius="1" length="1"/>
+      </geometry>
+      <material name="grey"/>
+    </visual>
+    <collision>
+      <origin xyz="0.0 0.0 0.0" rpy="0 0 0"/>
+      <geometry>
+        <cylinder radius="1" length="1"/>
+      </geometry>
+    </collision>
+    <inertial>
+      <origin xyz="3.0876154e-04 0.0000000e+00 -1.2176461e-04" />
+      <mass value="7.9119962e-02" />
+      <inertia ixx="1.2505234e-05" ixy="0.0" ixz="-1.7855208e-07"
+               iyy="2.1898364e-05" iyz="0.0"
+               izz="1.9267361e-05" />
+    </inertial>
+  </link>
+  <joint name="base_link_plate_joint" type="revolute">
+    <parent link="base_link"/>
+    <child link="child_link"/>
+    <origin xyz="0.0 0.0 2.5" rpy="0 0 0"/>
+    <axis xyz="0 0 1"/>
+    <limit velocity="4.8" effort="1" lower="${-pi*0.9}" upper="${pi*0.9}"/>
+  </joint>
 </robot>

Commit message: controllers

File: test_package/xacro/bot.xacro (robot description, xacro)
@@ -1,4 +1,11 @@
 <?xml version="1.0"?>
 <robot name="test_bot" xmlns:xacro="http://ros.org/wiki/xacro">
+  <!-- Base Footprint -->
+  <link name="base_footprint"/>
+  <joint name="base_joint" type="fixed">
+    <parent link="base_footprint"/>
+    <child link="base_link"/>
+    <origin xyz="0.0 0.0 0.5" rpy="0 0 0"/>
+  </joint>
   <!-- Base_Link -->
   <link name="base_link">
@@ -8,5 +15,5 @@
         <cylinder radius="1" length="1"/>
       </geometry>
-      <material name="grey"/>
+      <!-- <material name="grey"/> -->
     </visual>
     <collision>
@@ -18,5 +25,5 @@
     <inertial>
       <origin xyz="3.0876154e-04 0.0000000e+00 -1.2176461e-04" />
-      <mass value="7.9119962e-02" />
+      <mass value="1" />
       <inertia ixx="1.2505234e-05" ixy="0.0" ixz="-1.7855208e-07"
                iyy="2.1898364e-05" iyz="0.0"
@@ -30,5 +37,5 @@
         <cylinder radius="1" length="1"/>
       </geometry>
-      <material name="grey"/>
+      <!-- <material name="grey"/> -->
     </visual>
     <collision>
@@ -51,5 +58,29 @@
     <origin xyz="0.0 0.0 2.5" rpy="0 0 0"/>
     <axis xyz="0 0 1"/>
-    <limit velocity="4.8" effort="1" lower="${-pi*0.9}" upper="${pi*0.9}"/>
+    <limit velocity="4.8" effort="1" lower="1000" upper="1000"/>
   </joint>
+  <ros2_control name="IgnitionSystem" type="system">
+    <hardware>
+      <plugin>ign_ros2_control/IgnitionSystem</plugin>
+    </hardware>
+    <joint name="base_link_plate_joint">
+      <command_interface name="position">
+        <param name="min">1000</param>
+        <param name="max">1000</param>
+      </command_interface>
+      <state_interface name="position">
+        <param name="initial_value">0.0</param>
+      </state_interface>
+      <state_interface name="velocity"/>
+      <state_interface name="effort"/>
+    </joint>
+  </ros2_control>
+  <gazebo>
+    <plugin filename="ign_ros2_control-system" name="ign_ros2_control::IgnitionROS2ControlPlugin">
+      <robot_param>robot_description</robot_param>
+      <robot_param_node>robot_state_publisher</robot_param_node>
+      <parameters>$(find test_package)/config/controllers.yaml</parameters>
+      <controller_manager_name>controller_manager</controller_manager_name>
+    </plugin>
+  </gazebo>
 </robot>

Commit message: fix urdf joint limits

File: test_package/xacro/bot.xacro (robot description, xacro)
@@ -26,7 +26,7 @@
       <origin xyz="3.0876154e-04 0.0000000e+00 -1.2176461e-04" />
       <mass value="1" />
-      <inertia ixx="1.2505234e-05" ixy="0.0" ixz="-1.7855208e-07"
-               iyy="2.1898364e-05" iyz="0.0"
-               izz="1.9267361e-05" />
+      <inertia ixx="1.2505234e-02" ixy="0.0" ixz="-1.7855208e-07"
+               iyy="2.1898364e-02" iyz="0.0"
+               izz="1.9267361e-02" />
     </inertial>
   </link>
@@ -35,5 +35,6 @@
       <origin xyz="0 0 0"  rpy="0 0 0"/>
       <geometry>
-        <cylinder radius="1" length="1"/>
+        <!-- <cylinder radius="1" length="1"/> -->
+        <box size="1 1 1"/>
       </geometry>
       <!-- <material name="grey"/> -->
@@ -42,5 +43,6 @@
       <origin xyz="0.0 0.0 0.0" rpy="0 0 0"/>
       <geometry>
-        <cylinder radius="1" length="1"/>
+        <!-- <cylinder radius="1" length="1"/> -->
+        <box size="1 1 1"/>
       </geometry>
     </collision>
@@ -58,5 +60,5 @@
     <origin xyz="0.0 0.0 2.5" rpy="0 0 0"/>
     <axis xyz="0 0 1"/>
-    <limit velocity="4.8" effort="1" lower="1000" upper="1000"/>
+    <limit velocity="10" effort="100" lower="-1000" upper="1000"/>
   </joint>
   <ros2_control name="IgnitionSystem" type="system">
@@ -66,5 +68,5 @@
     <joint name="base_link_plate_joint">
       <command_interface name="position">
-        <param name="min">1000</param>
+        <param name="min">-1000</param>
         <param name="max">1000</param>
       </command_interface>
